File: solenoid.brd (EAGLE design)
At the start: 35.6 x 30.5 mm, 40 parts, among them U1 ULN2003V12, U2 ULN2003V12, Y1 ECS-80-S-4X

Commit message: uwu
Parts:
- moved R7 21.9 mm to (18.3, 7.44), turned to 90 degrees
- moved D1 21.5 mm to (16.0, 6.68)
- moved R10 18.6 mm to (5.66, 7.70), turned to 180 degrees
- moved R11 17.2 mm to (8.20, 8.56), turned to 270 degrees
- moved C11 15.6 mm to (10.0, 8.43)
- moved D4 14.2 mm to (15.9, 7.97)
- moved R4 13.9 mm to (12.6, 7.57)
- moved R6 13.8 mm to (12.6, 9.37)
- moved D2 13.7 mm to (15.9, 9.45)
- moved U$8 0.09 mm to (13.7, 14.8)
Routing:
- net 12V: track 0.00 -> 66.2 mm, vias 0 -> 1
- net SWDIO: track 0.00 -> 65.7 mm, vias 0 -> 2
- net +3V3: track 19.4 -> 81.3 mm
- net SOL4_2: track 0.00 -> 30.6 mm
- net SOL4_1: track 0.00 -> 24.2 mm, vias 0 -> 1
- net SOL2_2: track 0.00 -> 20.6 mm, vias 0 -> 1
- net SOL2_1: track 0.00 -> 20.4 mm
- net SOL6_2: track 0.00 -> 17.6 mm
- net SWCLK: track 0.00 -> 16.7 mm
- net GND: track 17.3 -> 34.0 mm, vias 0 -> 2
- net SOL5_2: track 0.00 -> 16.5 mm
- net SOL5_1: track 0.00 -> 15.8 mm
- net SOL6_1: track 0.00 -> 14.4 mm
- net GPIO8: track 0.00 -> 13.7 mm, vias 0 -> 1
- net SOL1_2: track 0.00 -> 13.2 mm
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
Commit message: k
Parts:
- removed U2: ULN2003V12, ULN2003V12:ULN2003V12
- moved U$8 10.5 mm to (5.71, 21.6), turned to 270 degrees
- moved C11 6.12 mm to (7.37, 13.9), turned to 180 degrees
- moved U1 5.91 mm to (15.8, 14.2), turned to 0 degrees
- moved R10 5.29 mm to (9.05, 11.8), turned to 0 degrees
- moved J4 4.19 mm to (5.66, 9.02), turned to 0 degrees
- moved R11 4.04 mm to (5.74, 11.8), turned to 0 degrees
- moved J3 3.07 mm to (2.67, 19.4)
- moved J7 0.95 mm to (3.02, 2.41)
- moved J8 0.79 mm to (6.00, 2.34)
- moved J5 0.77 mm to (2.78, 13.7)
- moved J6 0.77 mm to (2.77, 8.09)
- moved J2 0.61 mm to (8.95, 2.33)
- moved J1 0.33 mm to (11.9, 2.31)
Connections:
- removed net SOL1_2: J1.1, U1.13
- removed net SOL2_2: J2.1, U1.11
- removed net SOL3_2: J5.1, U2.15
- removed net SOL4_2: J6.1, U2.13
- removed net SOL5_2: J7.1, U2.11
- removed net SOL6_2: J8.1, U1.15
- new net GPIO4: U1.4
- new net GPIO5: U1.5
- new net GPIO6: U1.6
- net 12V: now also J1.1, J2.1, J5.1, J6.1, J7.1, J8.1; no longer U2.9
- net GND: no longer U2.8
- net GPIO0: no longer U1.6
- net GPIO1: now also U1.1; no longer U1.5
- net GPIO10: no longer U2.3
- net GPIO11: no longer U2.4
- net GPIO12: no longer U2.5
- net GPIO13: no longer U2.6
- net GPIO14: no longer U1.1
- net GPIO15: no longer U1.2
- net GPIO2: now also U1.2; no longer U1.4
- net GPIO8: no longer U2.1
- net GPIO9: no longer U2.2
- net SOL1_1: now also U1.16; no longer U1.14
- net SOL2_1: now also U1.15; no longer U1.12
- net SOL3_1: now also U1.14; no longer U2.16
- net SOL4_1: now also U1.13; no longer U2.14
- net SOL5_1: now also U1.12; no longer U2.12
- net SOL6_1: now also U1.11; no longer U1.16
Routing:
- net 12V: track 66.2 -> 21.9 mm
- net SWDIO: track 65.7 -> 23.6 mm, vias 2 -> 1
- net SOL4_2: track 30.6 -> 0.00 mm
- net SOL2_2: track 20.6 -> 0.00 mm, vias 1 -> 0
- net SOL6_2: track 17.6 -> 0.00 mm
- net SOL5_2: track 16.5 -> 0.00 mm
- net GPIO8: track 13.7 -> 0.00 mm, vias 1 -> 0
- net GND: track 34.0 -> 20.7 mm, vias 2 -> 11
- net CAN_RX: track 4.16 -> 17.4 mm, vias 0 -> 2
- net SOL1_2: track 13.2 -> 0.00 mm
- net SOL4_1: track 24.2 -> 12.3 mm, vias 1 -> 0
- net GPIO9: track 11.1 -> 0.00 mm, vias 1 -> 0
- net SOL3_2: track 10.9 -> 0.00 mm
- net GPIO10: track 10.1 -> 0.00 mm, vias 1 -> 0
- net GPIO11: track 9.54 -> 0.00 mm, vias 1 -> 0
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- added copper zone on layer 1, net 12V
- added copper zone on layer 1, net BA
- added copper zone on layer 16, net BA
- added copper zone on layer 1, net BAD
- added copper zone on layer 16, net BAD

Commit message: worked on some trace things and wiring
Parts:
- moved R2 1.63 mm to (33.6, 8.02), turned to 270 degrees
- moved C1 0.38 mm to (33.6, 6.29)
Routing:
- net +3V3: track 81.1 -> 102.9 mm
- net N$1: track 7.50 -> 9.79 mm
- net GND: track 20.7 -> 22.1 mm, vias 11 -> 21
- net CAN_RX: track 17.4 -> 18.0 mm
