File: solenoid.sch (EAGLE design)
At the start: 44 parts, among them Y1 ECS-80-S-4X

Commit message: Switched mosfets out for H-bridges
Deleted the solenoid mosfets and replaced them with 4 H-bridge parts

Signed-off-by: Callum Gundlach <gundlachcallum@gmail.com>
Parts:
- removed Q1, Q2, Q3, Q4, Q5, Q6, Q7, Q8: (no value), microbuilder:MOSFET-NWIDE
- added C18: 47uF, SparkFun-Capacitors:47UF-POLAR-PANASONIC_D-35V-20%
- added U$1, U$2, U$5, U$6: LV8548M, HBridge:LV8548M
Connections:
- removed net DRAIN0: J1.1, Q3.D
- removed net DRAIN1: J2.1, Q2.D
- removed net DRAIN2: J3.1, Q1.D
- removed net DRAIN3: J4.1, Q4.D
- removed net DRAIN4: J5.1, Q5.D
- removed net DRAIN5: J6.1, Q8.D
- removed net DRAIN6: J7.1, Q7.D
- removed net DRAIN7: J8.1, Q6.D
- new net GPIO10: U$3.PA5, U$5.IN3
- new net GPIO11: U$3.PA6, U$5.IN4
- new net GPIO12: U$3.PA7, U$6.IN1
- new net GPIO13: U$3.PA8, U$6.IN2
- new net GPIO14: U$3.PA9, U$6.IN3
- new net GPIO15: U$3.PA10, U$6.IN4
- new net GPIO8: U$3.PA3, U$5.IN1
- new net GPIO9: U$3.PA4, U$5.IN2
- new net SOL1_1: J1.2, U$1.OUT1
- new net SOL1_2: J1.1, U$1.OUT2
- new net SOL2_1: J2.2, U$1.OUT3
- new net SOL2_2: J2.1, U$1.OUT4
- new net SOL3_1: J3.2, U$2.OUT1
- new net SOL3_2: J3.1, U$2.OUT2
- new net SOL4_1: J4.2, U$2.OUT3
- new net SOL4_2: J4.1, U$2.OUT4
- new net SOL5_1: J5.2, U$5.OUT1
- new net SOL5_2: J5.1, U$5.OUT2
- new net SOL6_1: J6.2, U$5.OUT3
- new net SOL6_2: J6.1, U$5.OUT4
- new net SOL7_1: J7.2, U$6.OUT1
- new net SOL7_2: J7.1, U$6.OUT2
- new net SOL8_1: J8.2, U$6.OUT3
- new net SOL8_2: J8.1, U$6.OUT4
- net 12V: now also C18.+, U$1.VCC, U$2.VCC, U$5.VCC, U$6.VCC; no longer J1.2, J2.2, J3.2, J4.2, J5.2, J6.2, J7.2, J8.2
- net GND: now also C18.-, U$1.GND, U$2.GND, U$5.GND, U$6.GND; no longer Q1.S, Q2.S, Q3.S, Q4.S, Q5.S, Q6.S, Q7.S, Q8.S
- net GPIO0: now also U$1.IN1; no longer Q3.G
- net GPIO1: now also U$1.IN2; no longer Q2.G
- net GPIO2: now also U$1.IN3; no longer Q1.G
- net GPIO3: now also U$1.IN4; no longer Q4.G
- net GPIO4: now also U$2.IN1; no longer Q5.G
- net GPIO5: now also U$2.IN2; no longer Q8.G
- net GPIO6: now also U$2.IN3; no longer Q7.G
- net GPIO7: now also U$2.IN4; no longer Q6.G
Other:
- note added: "H-Bridges"
- note removed: "DMN67D8L-7DICT-ND"
- note removed: "MOSFETS"
- moved on the sheet: D2, D4, J1, J2, J3, J4, J5, J6, J7, J8, R4, R6

Commit message: Created the board and placed everything.  Started routing
Changed lines of the file:
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@@
 <part name="SUPPLY19" library="SparkFun-PowerSymbols" library_urn="urn:adsk.eagle:library:530" deviceset="12V" device=""/>
 <part name="C18" library="SparkFun-Capacitors" library_urn="urn:adsk.eagle:library:510" deviceset="47UF-POLAR" device="-PANASONIC_D-35V-20%" package3d_urn="urn:adsk.eagle:package:37420/1" value="47uF"/>
+<part name="+3V4" library="supply1" library_urn="urn:adsk.eagle:library:371" deviceset="+3V3" device=""/>
 </parts>
 <sheets>
@@
 <attribute name="NAME" x="122.936" y="59.055" size="1.778" layer="95" font="vector"/>
 <attribute name="VALUE" x="122.936" y="54.229" size="1.778" layer="96" font="vector"/>
+</instance>
+<instance part="+3V4" gate="G$1" x="317.5" y="147.32" smashed="yes">
+<attribute name="VALUE" x="314.96" y="142.24" size="1.778" layer="96" rot="R90"/>
 </instance>
 </instances>
@@
 </segment>
 <segment>
-<pinref part="U$3" gate="G$1" pin="VDD"/>
-<wire x1="332.74" y1="142.24" x2="317.5" y2="142.24" width="0.1524" layer="91"/>
-<label x="317.5" y="142.24" size="1.778" layer="95"/>
-</segment>
-<segment>
 <pinref part="U$3" gate="G$1" pin="VDDIO2"/>
 <wire x1="378.46" y1="121.92" x2="396.24" y2="121.92" width="0.1524" layer="91"/>
@@
 <label x="317.5" y="129.54" size="1.778" layer="95"/>
 </segment>
+<segment>
+<pinref part="U$3" gate="G$1" pin="VDD"/>
+<wire x1="332.74" y1="142.24" x2="317.5" y2="142.24" width="0.1524" layer="91"/>
+<pinref part="+3V4" gate="G$1" pin="+3V3"/>
+<wire x1="317.5" y1="144.78" x2="317.5" y2="142.24" width="0.1524" layer="91"/>
+</segment>
 </net>

Commit message: Newly sized board w/ schematic changes
This is the first attempt at routing the 1.2" by  1.4" solenoid board with a removed h-bridge and with some questions as to some airwires
Parts:
- removed J3, J4: (no value), SparkFun-Connectors:CONN_02
- removed U$2: LV8548M, HBridge:LV8548M
- added U$7: T2I, BackplaneParts:T2I
Connections:
- removed net GPIO4: U$2.IN1, U$3.PB5
- removed net GPIO5: U$2.IN2, U$3.PA0
- removed net GPIO6: U$2.IN3, U$3.PA1
- removed net GPIO7: U$2.IN4, U$3.PA2
- removed net SOL3_1: J3.2, U$2.OUT1
- removed net SOL3_2: J3.1, U$2.OUT2
- removed net SOL4_1: J4.2, U$2.OUT3
- removed net SOL4_2: J4.1, U$2.OUT4
- net 12V: now also U$7.3; no longer U$2.VCC
- net CAN_H: now also U$7.1
- net CAN_L: now also U$7.2
- net GND: now also U$7.4; no longer U$2.GND
- net GPIO0: now also U$1.IN4; no longer U$1.IN1
- net GPIO1: now also U$1.IN3; no longer U$1.IN2
- net GPIO2: now also U$1.IN2; no longer U$1.IN3
- net GPIO3: now also U$1.IN1; no longer U$1.IN4
Other:
- note added: "T21 Connector for 12V, CAN, GND"

Commit message: added new components
Connections:
- net GPIO0: now also U$1.IN1; no longer U$1.IN4
- net GPIO1: now also U$1.IN2; no longer U$1.IN3
- net GPIO2: now also U$1.IN3; no longer U$1.IN2
- net GPIO3: now also U$1.IN4; no longer U$1.IN1
Changed lines of the file:
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@@
 </segment>
 <segment>
-<pinref part="U$1" gate="G$1" pin="IN3"/>
-<wire x1="-2.54" y1="-48.26" x2="-12.7" y2="-48.26" width="0.1524" layer="91"/>
-<label x="-12.7" y="-48.26" size="1.778" layer="95"/>
+<pinref part="U$1" gate="G$1" pin="IN2"/>
+<wire x1="-2.54" y1="-43.18" x2="-12.7" y2="-43.18" width="0.1524" layer="91"/>
+<label x="-12.7" y="-43.18" size="1.778" layer="95"/>
 </segment>
 </net>
@@
 </segment>
 <segment>
-<pinref part="U$1" gate="G$1" pin="IN4"/>
-<wire x1="-2.54" y1="-53.34" x2="-12.7" y2="-53.34" width="0.1524" layer="91"/>
-<label x="-12.7" y="-53.34" size="1.778" layer="95"/>
+<pinref part="U$1" gate="G$1" pin="IN1"/>
+<wire x1="-2.54" y1="-38.1" x2="-12.7" y2="-38.1" width="0.1524" layer="91"/>
+<label x="-12.7" y="-38.1" size="1.778" layer="95"/>
 </segment>
 </net>
@@
 </segment>
 <segment>
-<pinref part="U$1" gate="G$1" pin="IN1"/>
-<wire x1="-2.54" y1="-38.1" x2="-12.7" y2="-38.1" width="0.1524" layer="91"/>
-<label x="-12.7" y="-38.1" size="1.778" layer="95"/>
+<pinref part="U$1" gate="G$1" pin="IN4"/>
+<wire x1="-2.54" y1="-53.34" x2="-12.7" y2="-53.34" width="0.1524" layer="91"/>
+<label x="-12.7" y="-53.34" size="1.778" layer="95"/>
 </segment>
 </net>
@@
 </segment>
 <segment>
-<pinref part="U$1" gate="G$1" pin="IN2"/>
-<wire x1="-2.54" y1="-43.18" x2="-12.7" y2="-43.18" width="0.1524" layer="91"/>
-<label x="-12.7" y="-43.18" size="1.778" layer="95"/>
+<pinref part="U$1" gate="G$1" pin="IN3"/>
+<wire x1="-2.54" y1="-48.26" x2="-12.7" y2="-48.26" width="0.1524" layer="91"/>
+<label x="-12.7" y="-48.26" size="1.778" layer="95"/>
 </segment>
 </net>
