File: solenoid.sch (EAGLE design)
At the start: 37 parts, among them Y1 ECS-80-S-4X

Commit message: owo
Parts:
- added U1, U2, U3, U4, U5, U6: QS5K2TR, QS5K2TR:QS5K2TR
Connections:
- net 12V: now also U1.TR1_TR2_SOURCE, U2.TR1_TR2_SOURCE, U3.TR1_TR2_SOURCE, U4.TR1_TR2_SOURCE, U5.TR1_TR2_SOURCE, U6.TR1_TR2_SOURCE
Changed lines of the file:
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@@
 <part name="J4" library="SparkFun-Connectors" library_urn="urn:adsk.eagle:library:513" deviceset="CONN_02" device="" package3d_urn="urn:adsk.eagle:package:38039/1"/>
 <part name="U$2" library="MURATA_3pin_dcdc" deviceset="MURATA-DC-DC" device="" package3d_urn="urn:adsk.eagle:package:23169699/2"/>
+<part name="U1" library="QS5K2TR" deviceset="QS5K2TR" device=""/>
+<part name="U2" library="QS5K2TR" deviceset="QS5K2TR" device=""/>
+<part name="U3" library="QS5K2TR" deviceset="QS5K2TR" device=""/>
+<part name="U4" library="QS5K2TR" deviceset="QS5K2TR" device=""/>
+<part name="U5" library="QS5K2TR" deviceset="QS5K2TR" device=""/>
+<part name="U6" library="QS5K2TR" deviceset="QS5K2TR" device=""/>
 </parts>
 <sheets>
@@
 <instance part="U$2" gate="G$1" x="167.64" y="63.5" smashed="yes">
 <attribute name="NAME" x="165.1" y="66.04" size="1.778" layer="95"/>
+</instance>
+<instance part="U1" gate="G$1" x="-2.54" y="-35.56" smashed="yes">
+<attribute name="VALUE" x="-10.16991875" y="-50.8198" size="1.78031875" layer="96"/>
+<attribute name="NAME" x="-10.17515" y="-21.8167" size="1.78153125" layer="95"/>
+</instance>
+<instance part="U2" gate="G$1" x="33.02" y="-35.56" smashed="yes">
+<attribute name="VALUE" x="25.39008125" y="-50.8198" size="1.78031875" layer="96"/>
+<attribute name="NAME" x="25.38485" y="-21.8167" size="1.78153125" layer="95"/>
+</instance>
+<instance part="U3" gate="G$1" x="-2.54" y="-88.9" smashed="yes">
+<attribute name="VALUE" x="-10.16991875" y="-104.1598" size="1.78031875" layer="96"/>
+<attribute name="NAME" x="-10.17515" y="-75.1567" size="1.78153125" layer="95"/>
+</instance>
+<instance part="U4" gate="G$1" x="33.02" y="-88.9" smashed="yes">
+<attribute name="VALUE" x="25.39008125" y="-104.1598" size="1.78031875" layer="96"/>
+<attribute name="NAME" x="25.38485" y="-75.1567" size="1.78153125" layer="95"/>
+</instance>
+<instance part="U5" gate="G$1" x="-2.54" y="-137.16" smashed="yes">
+<attribute name="VALUE" x="-10.16991875" y="-152.4198" size="1.78031875" layer="96"/>
+<attribute name="NAME" x="-10.17515" y="-123.4167" size="1.78153125" layer="95"/>
+</instance>
+<instance part="U6" gate="G$1" x="33.02" y="-137.16" smashed="yes">
+<attribute name="VALUE" x="25.39008125" y="-152.4198" size="1.78031875" layer="96"/>
+<attribute name="NAME" x="25.38485" y="-123.4167" size="1.78153125" layer="95"/>
 </instance>
 </instances>
@@
 <label x="411.48" y="-48.26" size="1.778" layer="95"/>
 </segment>
-</net>
+<segment>
+<pinref part="U1" gate="G$1" pin="TR1_TR2_SOURCE"/>
+<wire x1="-12.7" y1="-35.56" x2="-17.78" y2="-35.56" width="0.1524" layer="91"/>
+<label x="-22.86" y="-35.56" size="1.778" layer="95"/>
+</segment>
+<segment>
+<pinref part="U2" gate="G$1" pin="TR1_TR2_SOURCE"/>
+<wire x1="22.86" y1="-35.56" x2="17.78" y2="-35.56" width="0.1524" layer="91"/>
+<label x="12.7" y="-35.56" size="1.778" layer="95"/>
+</segment>
+<segment>
+<pinref part="U3" gate="G$1" pin="TR1_TR2_SOURCE"/>
+<wire x1="-12.7" y1="-88.9" x2="-17.78" y2="-88.9" width="0.1524" layer="91"/>
+<label x="-22.86" y="-88.9" size="1.778" layer="95"/>
+</segment>
+<segment>
+<pinref part="U4" gate="G$1" pin="TR1_TR2_SOURCE"/>
+<wire x1="22.86" y1="-88.9" x2="17.78" y2="-88.9" width="0.1524" layer="91"/>
+<label x="12.7" y="-88.9" size="1.778" layer="95"/>
+</segment>
+<segment>
+<pinref part="U5" gate="G$1" pin="TR1_TR2_SOURCE"/>
+<wire x1="-12.7" y1="-137.16" x2="-17.78" y2="-137.16" width="0.1524" layer="91"/>
+<label x="-22.86" y="-137.16" size="1.778" layer="95"/>
+</segment>
+<segment>
+<pinref part="U6" gate="G$1" pin="TR1_TR2_SOURCE"/>
+<wire x1="22.86" y1="-137.16" x2="17.78" y2="-137.16" width="0.1524" layer="91"/>
+<label x="12.7" y="-137.16" size="1.778" layer="95"/>
+</segment>
+</net>
